File: Station_PCB/RX_module.kicad_sch (KiCad schematic)
At the start: 5 parts, among them J1 Conn_01x19_Socket, J2 Conn_01x19_Socket, J3 Conn_01x08_Socket, J4 Conn_01x08_Socket, J5 Conn_01x04_Socket

Commit message: Mejora placa y la deja en una sola cara para impresion
Parts:
- removed J2: Conn_01x19_Socket, Connector_PinSocket_2.54mm:PinSocket_1x19_P2.54mm_Vertical, symbol Connector:Conn_01x19_Socket
- added J2-1: Conn_01x11_Socket, Connector_PinSocket_2.54mm:PinSocket_1x11_P2.54mm_Vertical, symbol Connector:Conn_01x11_Socket
- added J2-2: Conn_01x06_Socket, Connector_PinSocket_2.54mm:PinSocket_1x06_P2.54mm_Vertical, symbol Connector:Conn_01x06_Socket
Connections:
- net CS: now also J2-2.2 (Pin_2)
- net GND: now also J2-1.1 (Pin_1), J2-1.7 (Pin_7)
- net MISO: now also J2-1.8 (Pin_8)
- net MOSI: now also J2-1.2 (Pin_2)
- net SCK: now also J2-1.9 (Pin_9)
- net SCL: now also J5.3 (Pin_3), J2-1.3 (Pin_3); no longer J5.4 (Pin_4)
- net SDA: now also J5.4 (Pin_4), J2-1.6 (Pin_6); no longer J5.3 (Pin_3)
